File: keyboard_creator/blankproject/blank.kicad_pcb (KiCad board)
At the start: 2 copper layers, 0 parts

Commit message: More notes, updated README
Routing:
- added copper zone on F.Cu, net (none)
Other:
- board text added: "(1) Make liberal use of the F.Fab and B.Fab layers. Those should be used for documentation which you want to relay to your fab house. Component pinage"
- board text added: "(1) USB DATA TRACES: make sure to route them as short as possible, parallel to one another. Also learn to use the phase skew adjustment tool of KiCAD. Avoid"
- board text added: "(2) CRYSTAL TRACES: these are the highest frequency traces on the PCB and should be handled with extreme care. Always place the crystal extremely close to"
- board text added: "(2) Treat the silkscreen layers with very good care. Make sure that the component designators are minimally sized (1mm tall with 0.2mm trace width is advised),"
- board text added: "(3) BYPASS CAPACITORS: the precise function and nature of bypass (also called decoupling) capacitors is difficult to explain without higher knowledge in maths"
- board text added: "(3) KiCAD allows custom user layers. Use those to indicate screw hole anchors/sizes, plate markings, stabilizer orientation. Document everything because"
- board text added: "(4) If you want to share or open-source your design, be kind and make sure all your thought process or ideas are clearly documented and defined. Revising"
- board text added: "(5) Yes, documenting is boring. Everyone knows that, and yet everyone takes the time to do it because it saves you time and headaches down the line."
- board text added: "- If you are beggining on PCB design or are using a new fab, it might be wise to just use the values here for now"
- board text added: "- Manufacturing parameters might change in which case the tolerance values will change accordingly"
- board text added: "- Such values *should* be enough for keyboard PCBs"
- board text added: "- The values used are based on experience but should be manufacturable at low cost and accepted industry-wide"
- board text added: "- You can freely change these parameters around but make sure what those changes entail to, cost and production-wise"
- board text added: "0.15 (see [i])"
- board text added: "0.3 (see [iii])"
- board text added: "0.5 (see [iv])"
- board text added: "1:5 (see [v])"
- board text added: "1:6 (see [ii])"
- board text added: "A change in manufacturing parameters (layers and copper weight) will unequivocaly change the minimum values."
- board text added: "At the bottom-right of the page there is a copper polygon with the settings generally used for the Acheron Project. The values are tuned for general use, but"
- board text added: "Avoid using hatched-pattern copper pours. They have their reason to be, but not on keyboard PCBs. They are ugly (yeah, fight me) and don't do what we want them"
- board text added: "EXAMPLE COPPER POUR"
- board text added: "Elecrow offers {dblquote}standard PCB{dblquote} and {dblquote}advanced PCB{dblquote} services ([2]), while PCBWay offers {dblquote}normal difficulty{dblquote}, {dblquote}medium difficulty{dblquote} and {dblquote}high difficulty{dblquote} processes ([3])"
- board text added: "Even though keyboard PCB design is very forgiving in terms of the mistakes and errors you can make, there are some problems that are potentially PCB-breaking."
- board text added: "For clarification, read the NOTES ON TOLERANCES."
- board text added: "For the actual values, check references [1-3]."
- board text added: "In both manufacturers, the advanced settings have smaller tolerances and better manufacturing features but are significantly more expensive, specially"
- board text added: "It must also be kept in mind that, since the Acheron Project is heavily DIY-oriented, the tolerance settings used were the easiest or cheapest available. For instance,"
- board text added: "LEDs and level shifters. Treat bypass capacitors like you would a crystal: as close to the main device as possible and with short traces. Always look at"
- board text added: "NOTES"
- board text added: "OVERALL DESIGN RECOMMENDATIONS"
- board text added: "PCB design involves a lot of creativity and not everyone understands your codes and conventions. Take good care of documenting your PCB. Some tips:"
- board text added: "PLEASE READ"
- board text added: "REFERENCES"
- board text added: "Sharing your design and knowledge is one of the most fruitful and effective ways to learn design and gain knowledge. Look at other people's designs and frequently"
- board text added: "TLDR"
- board text added: "The first experience with PCB design is always very frustrating and overwhelming. There will be a lot of failed prototypes before you consider yourself a minimally"
- board text added: "The manufacturing tolerances used for PCBs in the Acheron Project are a way to uniformize the design settings of the projects. These settings were obtained using"
- board text added: "The most common problems for first-timers in keyboard PCB design are (1) USB data traces routing (2) crystal traces routing and (3) bypass capacitors placement"
- board text added: "The values and observations here listed consider a two-layer, 1 oz/ft2 PCB"
- board text added: "Therefore even for a 2-layer 1oz/ft2 PCB tolerances can be different for the {dblquote}advanced{dblquote} or {dblquote}high-difficulty{dblquote} settings."
- board text added: "Therefore, it must always be understood that a single body of uniform tolerances throughout a wide spectrum of projects is unfeasible due to the very nature"
- board text added: "Values also pertain to the cheapest setting on the referenced manufacturers."
- board text added: "You should read it all though"
- board text added: "[1] PCBWay manufacturing capabilities. Link: <https://www.pcbway.com/capabilities.html>. Last access august 21, 2021."
- board text added: "[2] JLCPCB manufacturing capabilities. Link: <https://jlcpcb.com/capabilities/Capabilities>. Last accessed august 21, 2021."
- board text added: "[3] Elecrow manufacturing capabilities. Link: <https://www.elecrow.com/download/quote/PCB_Specification_FAQ.pdf> . Last access august 21, 2021."
- board text added: "[4] Sanjeeb Mishra, Neeraj Kumar Singh, Vijayakrishnan Rousseau. System on Chip Interfaces for Low Power Design. Morgan Kaufmann, 2016. ISBN 9780128016305. Accessible via https://www.sciencedirect.com/science/article/pii/B9780128016305000104)"
- board text added: "[i] Official copper-copper clearances are 0.2mm but not exactly {dblquote}all copper{dblquote}. Pad-to-pad minimums are 0.5mm in the case of THT pads and 0.2mm for SMD pads."
- board text added: "[ii] The recommended ratio between silkscreen character height and its trace width so they are clearly legible."
- board text added: "[iii] The hole-to-copper clearance changes on occasion. For instance, via-to-track and NPTH-to-track clearance is 0.25mm but PTH-to-track is 0.3."
- board text added: "[iv] The distance of copper-to-edge is a big problem for fabs in designs where traces need to be close to certain slots or the edges, like keyboard PCBs with flex cuts"
- board text added: "[v] The 1:6 ratio for silkscreen is OK for large characters but can become unreadable to the naked eye on a 1mm character. A 1:5 ratio is recommended."
- board text added: "a PCB, much like a computer code or a maths test, requires knowledge that is either a convention or only the author knows."
- board text added: "adjustments can be made. Thermal spoke width and relief gap can be adjusted according to the thermal needs -- for THT components or connectors, it is"
- board text added: "and engineering. In layman's terms, bypass capacitors are placed to mitigate noise inherently present in digital circuits due to the natural inductance"
- board text added: "and polarity, values, designators, everything goes to make the fab's job easier -- and yours in the process."
- board text added: "and requirements of the different PCB projects. The values suggested here used in these files are only *recommendations* based on experience, having been"
- board text added: "and routing. In this order, they are the most problematic parts of designing a keyboard PCB and are the most frequent issues."
- board text added: "breaking and VIA'ing them as much as possible. If those are needed, do so in a simmetrical manner. If also possible, please read on differential pair"
- board text added: "communication (see [4], pages 331-344)."
- board text added: "datasheets, reference manuals and application notes which will generally inform how many capacitors are needed and their respective values and sizes."
- board text added: "denominator was found. These values should not be used often, but seldomly at the designer's discretion and in ultimate case. Their use will incurr in higher"
- board text added: "does not accompany its files; when someone looks at the PCB, component designators and polarities should be very clear and direct."
- board text added: "electronics and embedded systems is also recommended, but higher education in maths and engineering is absolutely not needed to be a DIY designer."
- board text added: "good PCB designer, and there is always something to learn. Since PCB design is a highly technical and skill-oriented field, it can sometimes looks as"
- board text added: "high-density designs etc) and are completely unnecessary for keyboard projects."
- board text added: "in the eventuality you want to make a revision or correction, all the information is in the files and not somewhere else buried deep down in emails"
- board text added: "mainly three manufacturers: PCBWay, Elecrow and JLCPCB (see their capabilities pages on references [1-3]). These are big players in the asian PCB manufacturing"
- board text added: "market and the tolerances practiced by them are accepted industry-wide; hence, the values used here should be enough for most manufacturers."
- board text added: "of traces and the switching characteristic of digital circuitry. Failure to properly place and route these capacitors can lead to inability of the digital circuits"
- board text added: "or Discord conversations."
- board text added: "recommended to use higher gaps (0.5mm will do the trick) to avoid bad solder joints."
- board text added: "some sorte of black magic. Do not stray from resilience. The best way to learn PCB design is designing. Some study in the fundamental aspects of"
- board text added: "talk to other designers. This ensures a collective knowledge is achieved both in hard and soft skills."
- board text added: "the MCU (in its vicinities) and if possible sharing the same ground (ideally islanded)."
- board text added: "to do here. Always use solid fills. The drawback is that they can make the PCB stiffer, so use flex cuts on the PCB."
- board text added: "to work properly. In the specific case of keyboard PCBs, there are plenty of digital circuits that need decoupling, mainly the microcontroller, RGB underglow"
- board text added: "used in a myriad of projects throughout the Acheron Project and in Gondolindrim's personal and professional projects."
- board text added: "visible. Also make sure that the silkscreen indicates the polarity of components either through arrows or symbols. Remember that the physical PCB"
- board text added: "when paired with PCB assembly services. Such settings are meant for more complex projects (high-speed or analog signal processing, finer electronic components,"
- board text removed: "0.15 (see [1])"
- board text removed: "0.3 (see [3])"
- board text removed: "0.5 (see [4])"
- board text removed: "1:5 (see [5])"
- board text removed: "1:6 (see [2])"
- board text removed: "A change in these parameters (layers and copper weight) will unequivocaly change the minimum values."
- board text removed: "The values and observations here listed consider a two-layer, 1 oz/ft2 PCB setting."
- board text removed: "[1] Official copper-copper clearances are 0.2mm but not exactly {dblquote}all copper{dblquote}. Pad-to-pad minimums are 0.5mm in the case of THT pads and 0.2mm for SMD pads."
- board text removed: "[2] The recommended ratio between silkscreen character height and its trace width so they are clearly legible."
- board text removed: "[3] The hole-to-copper clearance changes on occasion. For instance, via-to-track and NPTH-to-track clearance is 0.25mm but PTH-to-track is 0.3."
- board text removed: "[4] The distance of copper-to-edge is a big problem for fabs in designs where traces need to be close to certain slots or the edges, like keyboard PCBs with flex cuts"
- board text removed: "[5] The 1:6 ratio for silkscreen is OK for large characters but can become unreadable to the naked eye on a 1mm character. A 1:5 ratio is recommended."
- board text removed: "denominator was found. these values should not be used often, but seldomly at the designer's discretion and in ultimate case. Their use will incurr in higher"

Commit message: Add Seeedstudio capabilities references
Other:
- board text added: "Yes I know it's a lot of stuff but please read, it's important I promise"
- board text added: "[5] Seeedstudio manufacturing capabilities. Link: <https://support.seeedstudio.com/knowledgebase/articles/447362-fusion-pcb-specification> . Last accessed august 21, 2021."
Changed lines of the file:
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@@
+    (effects (font (size 1 1) (thickness 0.2)) (justify left))
+  )
+  (gr_text "Yes I know it's a lot of stuff but please read, it's important I promise" (at 321.6 -6) (layer "Cmts.User")
     (effects (font (size 1 1) (thickness 0.2)) (justify left))
   )
@@
     (effects (font (size 1 1) (thickness 0.2)) (justify left))
   )
+  (gr_text "[5] Seeedstudio manufacturing capabilities. Link: <https://support.seeedstudio.com/knowledgebase/articles/447362-fusion-pcb-specification> . Last accessed august 21, 2021." (at 300 232.5) (layer "Cmts.User")
+    (effects (font (size 1 1) (thickness 0.15)) (justify left))
+  )
   (gr_text "VIA HOLE:" (at 523 26) (layer "Cmts.User")
